File: pcb/infocard/infocard.kicad_sch (KiCad schematic)
At the start: 5 parts, among them U1 NT3H2111W0FHKH

Commit message: add everything else
Parts:
- D1: footprint LED_SMD:LED_1206_3216Metric_Pad1.42x1.75mm_HandSolder -> LED_SMD:LED_0805_2012Metric
Changed lines of the file:
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@@
 			)
 		)
-		(property "Footprint" "LED_SMD:LED_1206_3216Metric_Pad1.42x1.75mm_HandSolder"
+		(property "Footprint" "LED_SMD:LED_0805_2012Metric"
 			(at 133.35 115.57 0)
 			(effects
